File: EnvelopeRate.kicad_sch (KiCad schematic)
At the start: 0 parts

Commit message: Fin de création de tous les schémas - envelope.kicad_sch - EnvelopeRate.kicad_sch
git-svn-id: file:///D%5C00%20-%20Dev%20&%20Calculs%5CRepoTortoiseSVN_PCB%5CRevivalChips/branches/Discrete-AY-3-8910@28 8d7748af-fe70-f644-8493-3f4b7ec62ef1
Parts:
- added U100, U101, U102, U99: 74LS85, symbol 74xx:74LS85
- added U103: 74LS03, symbol 74xx:74LS03
- added U88, U91: 74LS273, symbol 74xx:74LS273
- added U95, U96: 74LS541, symbol 74xx:74LS541
- added U97, U98: 4040, symbol 4xxx:4040
Connections:
- new net: U100.4 (Ia>b), U99.5 (Oa>b)
- new net: U100.3 (Ia=b), U99.6 (Oa=b)
- new net: U100.2 (Ia<b), U99.7 (Oa<b)
- new net: U103.6, U97.11 (Reset), U98.11 (Reset)
- new net: U100.5 (Oa>b), U101.4 (Ia>b)
- new net: U100.6 (Oa=b), U101.3 (Ia=b)
- new net: U100.7 (Oa<b), U101.2 (Ia<b)
- new net: U101.5 (Oa>b), U102.4 (Ia>b)
- new net: U101.6 (Oa=b), U102.3 (Ia=b)
- new net: U101.7 (Oa<b), U102.2 (Ia<b)
- new net: U102.5 (Oa>b), U103.2
- new net CLK-256: U103.1, U97.10 (CLK)
- new net ClkEnv: U103.3, U103.5
- new net DA0: U88.3 (D0), U91.3 (D0), U95.18 (Y0), U96.18 (Y0)
- new net DA1: U88.4 (D1), U91.4 (D1), U95.17 (Y1), U96.17 (Y1)
- new net DA2: U88.7 (D2), U91.7 (D2), U95.16 (Y2), U96.16 (Y2)
- new net DA3: U88.8 (D3), U91.8 (D3), U95.15 (Y3), U96.15 (Y3)
- new net DA4: U88.13 (D4), U91.13 (D4), U95.14 (Y4), U96.14 (Y4)
- new net DA5: U88.14 (D5), U91.14 (D5), U95.13 (Y5), U96.13 (Y5)
- new net DA6: U88.17 (D6), U91.17 (D6), U95.12 (Y6), U96.12 (Y6)
- new net DA7: U88.18 (D7), U91.18 (D7), U95.11 (Y7), U96.11 (Y7)
- new net Nibble00_0: U88.2 (Q0), U95.2 (A0), U99.15 (A3)
- new net Nibble00_1: U88.5 (Q1), U95.3 (A1), U99.13 (A2)
- new net Nibble00_2: U88.6 (Q2), U95.4 (A2), U99.12 (A1)
- new net Nibble00_3: U88.9 (Q3), U95.5 (A3), U99.10 (A0)
- new net Nibble01_0: U100.15 (A3), U88.12 (Q4), U95.6 (A4)
- new net Nibble01_1: U100.13 (A2), U88.15 (Q5), U95.7 (A5)
- new net Nibble01_2: U100.12 (A1), U88.16 (Q6), U95.8 (A6)
- new net Nibble01_3: U100.10 (A0), U88.19 (Q7), U95.9 (A7)
- new net Nibble02_0: U97.9 (Q0), U99.1 (B3)
- new net Nibble02_1: U97.7 (Q1), U99.14 (B2)
- new net Nibble02_2: U97.6 (Q2), U99.11 (B1)
- new net Nibble02_3: U97.5 (Q3), U99.9 (B0)
- new net Nibble03_0: U100.1 (B3), U97.3 (Q4)
- new net Nibble03_1: U100.14 (B2), U97.2 (Q5)
- new net Nibble03_2: U100.11 (B1), U97.4 (Q6)
- new net Nibble03_3: U100.9 (B0), U97.13 (Q7), U98.10 (CLK)
- new net Nibble10_0: U101.15 (A3), U91.2 (Q0), U96.2 (A0)
- new net Nibble10_1: U101.13 (A2), U91.5 (Q1), U96.3 (A1)
- new net Nibble10_2: U101.12 (A1), U91.6 (Q2), U96.4 (A2)
- new net Nibble10_3: U101.10 (A0), U91.9 (Q3), U96.5 (A3)
- new net Nibble11_0: U102.15 (A3), U91.12 (Q4), U96.6 (A4)
- new net Nibble11_1: U102.13 (A2), U91.15 (Q5), U96.7 (A5)
- new net Nibble11_2: U102.12 (A1), U91.16 (Q6), U96.8 (A6)
- new net Nibble11_3: U102.10 (A0), U91.19 (Q7), U96.9 (A7)
- new net Nibble12_0: U101.1 (B3), U98.9 (Q0)
- new net Nibble12_1: U101.14 (B2), U98.7 (Q1)
- new net Nibble12_2: U101.11 (B1), U98.6 (Q2)
- new net Nibble12_3: U101.9 (B0), U98.5 (Q3)
- new net Nibble13_0: U102.1 (B3), U98.3 (Q4)
- new net Nibble13_1: U102.14 (B2), U98.2 (Q5)
- new net Nibble13_2: U102.11 (B1), U98.4 (Q6)
- new net Nibble13_3: U102.9 (B0), U98.13 (Q7)
- new net VCC: U100.16 (VCC), U101.16 (VCC), U102.16 (VCC), U103.14 (VCC), U88.20 (VCC), U91.20 (VCC), U95.20 (VCC), U96.20 (VCC), U97.16 (VDD), U98.16 (VDD), U99.16 (VCC), U99.3 (Ia=b)
- new net VSS: U100.8 (GND), U101.8 (GND), U102.8 (GND), U103.7 (GND), U88.10 (GND), U91.10 (GND), U95.10 (GND), U96.10 (GND), U97.8 (VSS), U98.8 (VSS), U99.2 (Ia<b), U99.4 (Ia>b), U99.8 (GND)
- new net ~{RES}: U103.4, U88.1 (~{Mr}), U91.1 (~{Mr})
- new net ~{RdEnvolope}-Coarse: U95.1 (G1), U95.19 (G2)
- new net ~{RdEnvolope}-Fine: U96.1 (G1), U96.19 (G2)
- new net ~{WrEnvolope}-Coarse: U88.11 (Cp)
- new net ~{WrEnvolope}-Fine: U91.11 (Cp)
- no-connect marks 0 -> 16
