File: ctrl_and_clk.kicad_sch (KiCad schematic)
At the start: 9 parts, among them U1 74LS273, U35 74LS10, U37 74LS138, U55 74LS05, U59 4040, U77 74LS09

Commit message: Fin de création de tous les schémas - envelope.kicad_sch - EnvelopeRate.kicad_sch
git-svn-id: file:///D%5C00%20-%20Dev%20&%20Calculs%5CRepoTortoiseSVN_PCB%5CRevivalChips/branches/Discrete-AY-3-8910@28 8d7748af-fe70-f644-8493-3f4b7ec62ef1
Parts:
- renumbered U59 to U56, U37 to U72, U37 to U73, U37 to U74, U37 to U75, U1 to U76
Other:
- note added: "BC1/BDIR ========= 0 / 0 = idle 1 / 0 = Read data 0 / 1 = write data 1 / 1 = address"
