File: envelope.kicad_sch (KiCad schematic)
At the start: 0 parts

Commit message: Fin de création de tous les schémas - envelope.kicad_sch - EnvelopeRate.kicad_sch
git-svn-id: file:///D%5C00%20-%20Dev%20&%20Calculs%5CRepoTortoiseSVN_PCB%5CRevivalChips/branches/Discrete-AY-3-8910@28 8d7748af-fe70-f644-8493-3f4b7ec62ef1
Parts:
- added U79: 74LS273, symbol 74xx:74LS273
- added U80, U83: 74LS112, symbol 74xx:74LS112
- added U84: 74LS541, symbol 74xx:74LS541
- added U85: 74LS74, symbol 74xx:74LS74
- added U86: 74LS191, symbol 74xx:74LS191
- added U87: 74LS09, symbol 74xx:74LS09
- added U89, U90: 74LS32, symbol 74xx:74LS32
- added U92: 74LS05, symbol 74xx:74LS05
- added U93: 74LS11, symbol 74xx:74LS11
- added U94: 74LS03, symbol 74xx:74LS03
Connections:
- new net: U86.12 (Tc), U92.5
- new net: U80.1 (C), U83.10 (~{S}), U83.4 (~{S}), U92.6
- new net: U87.8, U90.10
- new net: U87.6, U90.9
- new net: U80.2 (K), U80.3 (J), U93.12
- new net: U89.1, U93.8
- new net: U83.5 (Q), U85.2 (D), U93.9
- new net: U86.14 (Cp), U89.6
- new net: U80.5 (Q), U86.5 (D/U)
- new net: U89.3, U89.4
- new net: U89.5, U89.8
- new net: U80.15 (~{R}), U90.3
- new net: U83.15 (~{R}), U85.6 (~{Q})
- new net: U87.11, U89.9
- new net: U85.9 (Q), U87.12
- new net: U87.10, U90.5, U92.12
- new net: U87.3, U89.10
- new net: U83.9 (Q), U93.3
- new net: U85.12 (D), U87.2, U93.6
- new net: U80.4 (~{S}), U89.11
- new net Alt: U87.13, U90.8, U92.3, U93.11
- new net Alternate: U79.5 (Q1), U84.3 (A1), U87.4
- new net Attack: U79.6 (Q2), U84.4 (A2), U87.9, U89.12, U92.1
- new net ClkEnv: U85.11 (C), U85.3 (C), U89.2
- new net Continue: U79.9 (Q3), U84.5 (A3), U87.5, U92.13
- new net DA0: U79.3 (D0), U84.18 (Y0)
- new net DA1: U79.4 (D1), U84.17 (Y1)
- new net DA2: U79.7 (D2), U84.16 (Y2)
- new net DA3: U79.8 (D3), U84.15 (Y3)
- new net DA4: U84.14 (Y4)
- new net DA5: U84.13 (Y5)
- new net DA6: U84.12 (Y6)
- new net DA7: U84.11 (Y7)
- new net Envelope0: U86.3 (Q0)
- new net Envelope1: U86.2 (Q1)
- new net Envelope2: U86.6 (Q2)
- new net Envelope3: U86.7 (Q3)
- new net Hold: U79.2 (Q0), U84.2 (A0), U90.4, U90.6, U92.11, U93.4
- new net Trig: U92.9, U94.3
- new net VCC: U79.20 (VCC), U80.10 (~{S}), U80.14 (~{R}), U80.16 (VCC), U83.16 (VCC), U84.20 (VCC), U85.1 (~{R}), U85.10 (~{S}), U85.13 (~{R}), U85.14 (VCC), U85.4 (~{S}), U86.16 (VCC), U87.14 (VCC), U89.14 (VCC), U90.14 (VCC), U92.14 (VCC), U93.14 (VCC), U93.2, U94.14 (VCC)
- new net VSS: U79.10 (GND), U79.13 (D4), U79.14 (D5), U79.17 (D6), U79.18 (D7), U80.11 (J), U80.12 (K), U80.13 (C), U80.8 (GND), U83.1 (C), U83.11 (J), U83.12 (K), U83.13 (C), U83.2 (K), U83.3 (J), U83.8 (GND), U84.10 (GND), U84.6 (A4), U84.7 (A5), U84.8 (A6), U84.9 (A7), U85.7 (GND), U86.4 (Ce), U86.8 (GND), U87.7 (GND), U89.7 (GND), U90.7 (GND), U92.7 (GND), U93.7 (GND), U94.7 (GND)
- new net ~{Alt}: U87.1, U92.4, U93.1
- new net ~{Attack}: U86.1 (P1), U86.10 (P2), U86.15 (P0), U86.9 (P3), U90.2, U92.2
- new net ~{Hold}: U92.10, U93.10, U93.13
- new net ~{RES}: U79.1 (~{Mr}), U94.2
- new net ~{RdEnvShape}: U84.1 (G1), U84.19 (G2)
- new net ~{Trig}: U83.14 (~{R}), U86.11 (Pl), U89.13, U90.1, U92.8, U93.5
- new net ~{WrEnvShape}: U79.11 (Cp), U94.1
- no-connect marks 0 -> 24
Other:
- note added: "AT AL HO ---------- 0 . 0 . 0 Falling sawtooth 0 . 0 . 1 Fall & stop 0 . 1 . 0 Falling triangle 0 . 1 . 1 Fall & Jump top 1 . 0 . 0 Rising Sawtooth 1 . 0 . 1 Rise & stop 1 . 1 . 0 Rising triangle 1 . 1 . 1 Rise & Jump zero if Continue==0 0xx -> 001 1xx -> 111"
